File: design/board.kicad_pcb (KiCad board)
At the start: 2 copper layers, 165 x 54 mm, 22 parts, among them J1 Conn_01x04_Male, J2 Conn_01x03_Male, J3 Conn_02x14_Odd_Even, J4 Conn_02x12_Odd_Even, SW1 reset, U1 W65C02_PLCC_44, U2 AT28C256_PDIP_28, U3 SRAM, U4 74LS00, U5 2-AND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

Commit message: gitignore.
Other:
- board text added: "#DMA"
- board text added: "Address Decoding"
- board text added: "CLK"
- board text added: "CLK I/O"
- board text added: "CPU"
- board text added: "CTRL"
- board text added: "GND"
- board text added: "I/O ports"
- board text added: "PWR"
- board text added: "PWR I/O"
- board text added: "RAM"
- board text added: "RESET"
- board text added: "ROM"
- board text added: "VCC"
- board text added: "Versatile Interface Adapater"
- board text added: "a0"
- board text added: "addr I/O"
- board text added: "d0"
- board text added: "d1"
- board text added: "d2"
- board text added: "d3"
- board text added: "d4"
- board text added: "d5"
- board text added: "d6"
- board text added: "d7"
- board text added: "data I/O"
Changed lines of the file:
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@@
   (general
     (thickness 1.6)
-    (drawings 4)
+    (drawings 62)
     (tracks 1217)
     (zones 0)
@@
   (layers
     (0 F.Cu signal)
-    (31 B.Cu signal)
+    (31 B.Cu signal hide)
     (32 B.Adhes user hide)
     (33 F.Adhes user hide)
@@
   )
   (setup
-    (last_trace_width 0.8)
+    (last_trace_width 0.5)
     (user_trace_width 0.2)
     (user_trace_width 0.25)
@@
       (layerselection 0x010fc_ffffffff)
       (usegerberextensions false)
-      (usegerberattributes false)
+      (usegerberattributes true)
       (usegerberadvancedattributes false)
       (creategerberjobfile false)
@@
       (plotinvisibletext false)
       (padsonsilk false)
-      (subtractmaskfromsilk false)
+      (subtractmaskfromsilk true)
       (outputformat 1)
       (mirror false)
-      (drillshape 1)
+      (drillshape 0)
       (scaleselection 1)
-      (outputdirectory ""))
+      (outputdirectory "/home/antoine/Documents/electronics/uComputer-mother-board/gerber/"))
   )
   (net 0 "")
@@
     (descr "Through hole straight socket strip, 2x14, 2.54mm pitch, double cols (from Kicad 4.0.7), script generated")
     (tags "Through hole socket strip THT 2x14 2.54mm double row")
-    (fp_text reference J3 (at -1.27 -2.77 90) (layer F.SilkS)
+    (fp_text reference J3 (at -1.27 16.51 180) (layer F.SilkS)
       (effects (font (size 1 1) (thickness 0.15)))
     )
@@
     (descr "Through hole straight pin header, 2x02, 2.54mm pitch, double rows")
     (tags "Through hole pin header THT 2x02 2.54mm double row")
-    (fp_text reference J1 (at 1.27 -2.33) (layer F.SilkS)
+    (fp_text reference J1 (at 1.27 1.27) (layer F.SilkS)
       (effects (font (size 1 1) (thickness 0.15)))
     )
@@
     (descr "Through hole straight pin header, 1x03, 2.54mm pitch, single row")
     (tags "Through hole pin header THT 1x03 2.54mm single row")
-    (fp_text reference J2 (at 0 -2.33) (layer F.SilkS)
+    (fp_text reference J2 (at 0 7.366) (layer F.SilkS)
       (effects (font (size 1 1) (thickness 0.15)))
     )
@@
   (module my_logic:SC-74A_p0.95 (layer F.Cu)
     (at 86.106 77.851 90)
-    (fp_text reference U5 (at 0.12 -0.72 90) (layer F.SilkS)
+    (fp_text reference U5 (at -0.381 -0.72 90) (layer F.SilkS)
       (effects (font (size 1 1) (thickness 0.15)))
     )
@@
     (at 39.37 53.594 90)
     (tags "socket Socket SOCKET PLCC DIP44 TH 1.27mm")
-    (fp_text reference U6 (at -2.667 6.54 180) (layer F.SilkS)
+    (fp_text reference U6 (at -1.397 6.223 180) (layer F.SilkS)
       (effects (font (size 1 1) (thickness 0.15)))
     )
@@
     (at 78.867 61.214 180)
     (tags "socket Socket SOCKET PLCC DIP44 TH 1.27mm")
-    (fp_text reference U1 (at -1.46 6.54) (layer F.SilkS)
+    (fp_text reference U1 (at -1.46 6.35) (layer F.SilkS)
       (effects (font (size 1 1) (thickness 0.15)))
     )
@@
     (descr "Through hole angled socket strip, 2x12, 2.54mm pitch, 8.51mm socket length, double cols (from Kicad 4.0.7), script generated")
     (tags "Through hole angled socket strip THT 2x12 2.54mm double row")
-    (fp_text reference J4 (at -9.271 15.113 180) (layer F.SilkS)
+    (fp_text reference J4 (at -8.636 13.97 180) (layer F.SilkS)
       (effects (font (size 1 1) (thickness 0.15)))
     )
@@
   (module my_buttons:pushbutton_button (layer F.Cu)
     (at 109.8595 79.5933)
-    (fp_text reference SW1 (at 0.381 0.889 180) (layer F.SilkS)
+    (fp_text reference SW1 (at 0.1225 -1.1073 180) (layer F.SilkS)
       (effects (font (size 1 1) (thickness 0.15)))
     )
@@
       (net 67 /GND))
   )
+  (gr_line (start 149.098 74.549) (end 151.13 74.549) (layer F.SilkS) (width 0.12))
+  (gr_line (start 138.811 74.549) (end 148.59 74.549) (layer F.SilkS) (width 0.12))
+  (gr_line (start 151.638 74.549) (end 153.67 74.549) (layer F.SilkS) (width 0.12))
+  (gr_line (start 154.178 74.549) (end 173.99 74.549) (layer F.SilkS) (width 0.12))
+  (gr_text a0 (at 172.974 75.057) (layer F.SilkS)
+    (effects (font (size 0.5 0.5) (thickness 0.125)))
+  )
+  (gr_text a0 (at 170.434 75.057) (layer F.SilkS)
+    (effects (font (size 0.5 0.5) (thickness 0.125)))
+  )
+  (gr_text a0 (at 167.894 75.057) (layer F.SilkS)
+    (effects (font (size 0.5 0.5) (thickness 0.125)))
+  )
+  (gr_text a0 (at 165.354 75.057) (layer F.SilkS)
+    (effects (font (size 0.5 0.5) (thickness 0.125)))
+  )
+  (gr_text a0 (at 162.814 75.057) (layer F.SilkS)
+    (effects (font (size 0.5 0.5) (thickness 0.125)))
+  )
+  (gr_text a0 (at 160.274 75.057) (layer F.SilkS)
+    (effects (font (size 0.5 0.5) (thickness 0.125)))
+  )
+  (gr_text a0 (at 157.734 75.057) (layer F.SilkS)
+    (effects (font (size 0.5 0.5) (thickness 0.125)))
+  )
+  (gr_text a0 (at 155.194 75.057) (layer F.SilkS)
+    (effects (font (size 0.5 0.5) (thickness 0.125)))
+  )
+  (gr_text a0 (at 155.194 81.153) (layer F.SilkS)
+    (effects (font (size 0.5 0.5) (thickness 0.125)))
+  )
+  (gr_text a0 (at 157.734 81.153) (layer F.SilkS)
+    (effects (font (size 0.5 0.5) (thickness 0.125)))
+  )
+  (gr_text a0 (at 160.274 81.153) (layer F.SilkS)
+    (effects (font (size 0.5 0.5) (thickness 0.125)))
+  )
+  (gr_text a0 (at 162.814 81.153) (layer F.SilkS)
+    (effects (font (size 0.5 0.5) (thickness 0.125)))
+  )
+  (gr_text a0 (at 165.354 81.153) (layer F.SilkS)
+    (effects (font (size 0.5 0.5) (thickness 0.125)))
+  )
+  (gr_text a0 (at 167.894 81.153) (layer F.SilkS)
+    (effects (font (size 0.5 0.5) (thickness 0.125)))
+  )
+  (gr_text a0 (at 170.434 81.153) (layer F.SilkS)
+    (effects (font (size 0.5 0.5) (thickness 0.125)))
+  )
+  (gr_text a0 (at 172.974 81.153) (layer F.SilkS)
+    (effects (font (size 0.5 0.5) (thickness 0.125)))
+  )
+  (gr_text d7 (at 139.954 75.057) (layer F.SilkS)
+    (effects (font (size 0.5 0.5) (thickness 0.125)))
+  )
+  (gr_text d5 (at 142.494 75.057) (layer F.SilkS)
+    (effects (font (size 0.5 0.5) (thickness 0.125)))
+  )
+  (gr_text d3 (at 145.034 75.057) (layer F.SilkS)
+    (effects (font (size 0.5 0.5) (thickness 0.125)))
+  )
+  (gr_text d1 (at 147.574 75.057) (layer F.SilkS)
+    (effects (font (size 0.5 0.5) (thickness 0.125)))
+  )
+  (gr_text "d6\n" (at 139.954 81.153) (layer F.SilkS)
+    (effects (font (size 0.5 0.5) (thickness 0.125)))
+  )
+  (gr_text d4 (at 142.494 81.153) (layer F.SilkS)
+    (effects (font (size 0.5 0.5) (thickness 0.125)))
+  )
+  (gr_text "d2\n" (at 145.034 81.153) (layer F.SilkS)
+    (effects (font (size 0.5 0.5) (thickness 0.125)))
+  )
+  (gr_text d0 (at 147.574 81.153) (layer F.SilkS)
+    (effects (font (size 0.5 0.5) (thickness 0.125)))
+  )
+  (gr_line (start 146.304 78.105) (end 148.844 78.105) (layer F.SilkS) (width 0.12))
+  (gr_line (start 146.304 80.645) (end 146.304 78.105) (layer F.SilkS) (width 0.12))
+  (gr_text GND (at 152.654 75.057) (layer F.SilkS)
+    (effects (font (size 0.5 0.5) (thickness 0.125)))
+  )
+  (gr_text VCC (at 152.654 81.153) (layer F.SilkS)
+    (effects (font (size 0.5 0.5) (thickness 0.125)))
+  )
+  (gr_line (start 154.178 81.661) (end 173.99 81.661) (layer F.SilkS) (width 0.12))
+  (gr_line (start 151.638 81.661) (end 153.67 81.661) (layer F.SilkS) (width 0.12))
+  (gr_line (start 149.098 81.661) (end 151.13 81.661) (layer F.SilkS) (width 0.12))
+  (gr_line (start 138.811 81.661) (end 148.59 81.661) (layer F.SilkS) (width 0.12))
+  (gr_text "#DMA" (at 150.114 75.057) (layer F.SilkS)
+    (effects (font (size 0.5 0.5) (thickness 0.125)))
+  )
+  (gr_text CLK (at 150.114 81.153) (layer F.SilkS)
+    (effects (font (size 0.5 0.5) (thickness 0.125)))
+  )
+  (gr_line (start 153.924 80.645) (end 153.924 75.565) (layer F.SilkS) (width 0.12))
+  (gr_line (start 151.384 80.645) (end 151.384 75.565) (layer F.SilkS) (width 0.12))
+  (gr_line (start 148.844 75.565) (end 148.844 80.645) (layer F.SilkS) (width 0.12))
+  (gr_text "addr I/O" (at 164.084 82.677) (layer F.SilkS)
+    (effects (font (size 1 1) (thickness 0.15)))
+  )
+  (gr_text PWR (at 152.654 83.566 90) (layer F.SilkS)
+    (effects (font (size 1 1) (thickness 0.15)))
+  )
+  (gr_text CTRL (at 150.114 83.566 90) (layer F.SilkS)
+    (effects (font (size 1 1) (thickness 0.15)))
+  )
+  (gr_text "data I/O" (at 143.764 82.677) (layer F.SilkS)
+    (effects (font (size 1 1) (thickness 0.15)))
+  )
+  (gr_text "PWR I/O" (at 133.604 82.042) (layer F.SilkS)
+    (effects (font (size 1 1) (thickness 0.15)))
+  )
+  (gr_text RESET (at 109.982 85.344) (layer F.SilkS)
+    (effects (font (size 2 2) (thickness 0.3)))
+  )
+  (gr_text "CLK I/O" (at 66.167 78.613 90) (layer F.SilkS)
+    (effects (font (size 1 1) (thickness 0.15)))
+  )
+  (gr_line (start 72.898 83.947) (end 72.898 72.644) (layer F.SilkS) (width 0.12))
+  (gr_line (start 88.392 83.947) (end 72.898 83.947) (layer F.SilkS) (width 0.12))
+  (gr_line (start 88.392 72.644) (end 88.392 83.947) (layer F.SilkS) (width 0.12))
+  (gr_line (start 72.898 72.644) (end 88.392 72.644) (layer F.SilkS) (width 0.12))
+  (gr_text "Address Decoding" (at 81.28 85.09) (layer F.SilkS)
+    (effects (font (size 1 1) (thickness 0.15)))
+  )
+  (gr_text ROM (at 137.16 53.086 90) (layer F.SilkS)
+    (effects (font (size 1 1) (thickness 0.15)))
+  )
+  (gr_text RAM (at 99.06 53.086 90) (layer F.SilkS)
+    (effects (font (size 1 1) (thickness 0.15)))
+  )
+  (gr_text "I/O ports" (at 29.21 79.502 90) (layer F.SilkS)
+    (effects (font (size 1 1) (thickness 0.15)))
+  )
+  (gr_text "Versatile Interface Adapater" (at 33.02 54.737 90) (layer F.SilkS)
+    (effects (font (size 1 1) (thickness 0.15)))
+  )
+  (gr_text CPU (at 67.31 53.721 90) (layer F.SilkS)
+    (effects (font (size 1 1) (thickness 0.15)))
+  )
   (gr_line (start 188.73 89.27) (end 23.73 89.27) (layer Edge.Cuts) (width 0.05))

Commit message: Silk for I/O ports.
Other:
- board text added: "GND in"
- board text added: "GND out"
- board text added: "VCC in"
- board text added: "VCC out"
- board text added: "a1"
- board text added: "a10"
- board text added: "a11"
- board text added: "a12"
- board text added: "a13"
- board text added: "a14"
- board text added: "a15"
- board text added: "a2"
- board text added: "a3"
- board text added: "a4"
- board text added: "a5"
- board text added: "a6"
- board text added: "a7"
- board text added: "a8"
- board text added: "a9"
- board text added: "ca1"
- board text added: "ca2"
- board text added: "cb1"
- board text added: "cb2"
- board text added: "pa0"
- board text added: "pa1"
- board text added: "pa2"
- board text added: "pa3"
- board text added: "pa4"
- board text added: "pa5"
- board text added: "pa6"
- board text added: "pa7"
- board text added: "pb0"
- board text added: "pb1"
- board text added: "pb2"
- board text added: "pb3"
- board text added: "pb4"
- board text added: "pb5"
- board text added: "pb6"
- board text added: "pb7"
Changed lines of the file:
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@@
   (general
     (thickness 1.6)
-    (drawings 62)
+    (drawings 106)
     (tracks 1217)
     (zones 0)
@@
   (layers
     (0 F.Cu signal)
-    (31 B.Cu signal hide)
+    (31 B.Cu signal)
     (32 B.Adhes user hide)
     (33 F.Adhes user hide)
@@
     (36 B.SilkS user)
     (37 F.SilkS user)
-    (38 B.Mask user hide)
+    (38 B.Mask user)
     (39 F.Mask user hide)
     (40 Dwgs.User user hide)
@@
   )
   (setup
-    (last_trace_width 0.5)
+    (last_trace_width 0.2)
     (user_trace_width 0.2)
     (user_trace_width 0.25)
@@
     (tags resistor)
     (attr smd)
-    (fp_text reference R3 (at 0 1.82 90) (layer B.SilkS)
+    (fp_text reference R3 (at -0.003 2.032 180) (layer B.SilkS)
       (effects (font (size 1 1) (thickness 0.15)) (justify mirror))
     )
@@
     (tags "capacitor handsolder")
     (attr smd)
-    (fp_text reference C5 (at 0 1.82 90) (layer B.SilkS)
+    (fp_text reference C5 (at 0 2.032 180) (layer B.SilkS)
       (effects (font (size 1 1) (thickness 0.15)) (justify mirror))
     )
@@
     (tags "capacitor handsolder")
     (attr smd)
-    (fp_text reference C4 (at 0 1.82 270) (layer B.SilkS)
+    (fp_text reference C4 (at 0 2.032) (layer B.SilkS)
       (effects (font (size 1 1) (thickness 0.15)) (justify mirror))
     )
@@
       (net 67 /GND))
   )
+  (gr_text "VCC\n" (at 70.612 76.073 270) (layer F.SilkS)
+    (effects (font (size 0.5 0.5) (thickness 0.125)))
+  )
+  (gr_line (start 71.12 75.057) (end 71.12 77.089) (layer F.SilkS) (width 0.12))
+  (gr_text CLK (at 70.612 81.153 270) (layer F.SilkS)
+    (effects (font (size 0.5 0.5) (thickness 0.125)))
+  )
+  (gr_line (start 71.12 80.137) (end 71.12 82.169) (layer F.SilkS) (width 0.12))
+  (gr_text GND (at 70.612 78.613 270) (layer F.SilkS)
+    (effects (font (size 0.5 0.5) (thickness 0.125)))
+  )
+  (gr_line (start 71.12 77.597) (end 71.12 79.629) (layer F.SilkS) (width 0.12))
+  (gr_text pb2 (at 52.07 85.979) (layer F.SilkS)
+    (effects (font (size 0.5 0.5) (thickness 0.125)))
+  )
+  (gr_text "VCC\n" (at 59.69 85.979) (layer F.SilkS)
+    (effects (font (size 0.5 0.5) (thickness 0.125)))
+  )
+  (gr_text "pb6\n" (at 46.99 85.979) (layer F.SilkS)
+    (effects (font (size 0.5 0.5) (thickness 0.125)))
+  )
+  (gr_text pb5 (at 49.53 87.122) (layer F.SilkS)
+    (effects (font (size 0.5 0.5) (thickness 0.125)))
+  )
+  (gr_text "GND\n" (at 59.69 87.122) (layer F.SilkS)
+    (effects (font (size 0.5 0.5) (thickness 0.125)))
+  )
+  (gr_text pb4 (at 49.53 85.979) (layer F.SilkS)
+    (effects (font (size 0.5 0.5) (thickness 0.125)))
+  )
+  (gr_text pb3 (at 52.07 87.122) (layer F.SilkS)
+    (effects (font (size 0.5 0.5) (thickness 0.125)))
+  )
+  (gr_text "pb0\n" (at 57.15 85.979) (layer F.SilkS)
+    (effects (font (size 0.5 0.5) (thickness 0.125)))
+  )
+  (gr_text cb2 (at 54.61 87.122) (layer F.SilkS)
+    (effects (font (size 0.5 0.5) (thickness 0.125)))
+  )
+  (gr_line (start 58.674 87.63) (end 60.706 87.63) (layer F.SilkS) (width 0.12))
+  (gr_line (start 58.674 85.471) (end 60.706 85.471) (layer F.SilkS) (width 0.12))
+  (gr_line (start 45.974 85.471) (end 58.039 85.471) (layer F.SilkS) (width 0.12))
+  (gr_line (start 45.974 87.63) (end 58.039 87.63) (layer F.SilkS) (width 0.12))
+  (gr_text cb1 (at 54.61 85.979) (layer F.SilkS)
+    (effects (font (size 0.5 0.5) (thickness 0.125)))
+  )
+  (gr_text pb7 (at 46.99 87.122) (layer F.SilkS)
+    (effects (font (size 0.5 0.5) (thickness 0.125)))
+  )
+  (gr_text pb1 (at 57.15 87.122) (layer F.SilkS)
+    (effects (font (size 0.5 0.5) (thickness 0.125)))
+  )
+  (gr_text "pa1\n" (at 34.29 87.122) (layer F.SilkS)
+    (effects (font (size 0.5 0.5) (thickness 0.125)))
+  )
+  (gr_text pa2 (at 39.37 85.979) (layer F.SilkS)
+    (effects (font (size 0.5 0.5) (thickness 0.125)))
+  )
+  (gr_text "GND\n" (at 31.75 87.122) (layer F.SilkS)
+    (effects (font (size 0.5 0.5) (thickness 0.125)))
+  )
+  (gr_text ca1 (at 36.83 85.979) (layer F.SilkS)
+    (effects (font (size 0.5 0.5) (thickness 0.125)))
+  )
+  (gr_text pa3 (at 39.37 87.122) (layer F.SilkS)
+    (effects (font (size 0.5 0.5) (thickness 0.125)))
+  )
+  (gr_text pa6 (at 44.45 85.979) (layer F.SilkS)
+    (effects (font (size 0.5 0.5) (thickness 0.125)))
+  )
+  (gr_text pa0 (at 34.29 85.979) (layer F.SilkS)
+    (effects (font (size 0.5 0.5) (thickness 0.125)))
+  )
+  (gr_text pa4 (at 41.91 85.979) (layer F.SilkS)
+    (effects (font (size 0.5 0.5) (thickness 0.125)))
+  )
+  (gr_text pa7 (at 44.45 87.122) (layer F.SilkS)
+    (effects (font (size 0.5 0.5) (thickness 0.125)))
+  )
+  (gr_text "VCC\n" (at 31.75 85.979) (layer F.SilkS)
+    (effects (font (size 0.5 0.5) (thickness 0.125)))
+  )
+  (gr_line (start 33.274 85.471) (end 45.466 85.471) (layer F.SilkS) (width 0.12))
+  (gr_line (start 33.274 87.63) (end 45.466 87.63) (layer F.SilkS) (width 0.12))
+  (gr_text "ca2\n" (at 36.83 87.122) (layer F.SilkS)
+    (effects (font (size 0.5 0.5) (thickness 0.125)))
+  )
+  (gr_line (start 30.734 85.471) (end 32.766 85.471) (layer F.SilkS) (width 0.12))
+  (gr_line (start 30.734 87.63) (end 32.766 87.63) (layer F.SilkS) (width 0.12))
+  (gr_text pa5 (at 41.91 87.122) (layer F.SilkS)
+    (effects (font (size 0.5 0.5) (thickness 0.125)))
+  )
+  (gr_text "GND out\n" (at 131.826 75.057) (layer F.SilkS)
+    (effects (font (size 0.5 0.5) (thickness 0.125)))
+  )
+  (gr_text "VCC out" (at 135.382 75.057) (layer F.SilkS)
+    (effects (font (size 0.5 0.5) (thickness 0.125)))
+  )
+  (gr_line (start 131.191 74.549) (end 136.017 74.549) (layer F.SilkS) (width 0.12))
+  (gr_line (start 131.191 81.661) (end 136.017 81.661) (layer F.SilkS) (width 0.12))
+  (gr_text "GND in" (at 131.826 81.153) (layer F.SilkS)
+    (effects (font (size 0.5 0.5) (thickness 0.125)))
+  )
+  (gr_text "VCC in" (at 135.382 81.153) (layer F.SilkS)
+    (effects (font (size 0.5 0.5) (thickness 0.125)))
+  )
   (gr_line (start 149.098 74.549) (end 151.13 74.549) (layer F.SilkS) (width 0.12))
   (gr_line (start 138.811 74.549) (end 148.59 74.549) (layer F.SilkS) (width 0.12))
   (gr_line (start 151.638 74.549) (end 153.67 74.549) (layer F.SilkS) (width 0.12))
   (gr_line (start 154.178 74.549) (end 173.99 74.549) (layer F.SilkS) (width 0.12))
-  (gr_text a0 (at 172.974 75.057) (layer F.SilkS)
-    (effects (font (size 0.5 0.5) (thickness 0.125)))
-  )
-  (gr_text a0 (at 170.434 75.057) (layer F.SilkS)
-    (effects (font (size 0.5 0.5) (thickness 0.125)))
-  )
-  (gr_text a0 (at 167.894 75.057) (layer F.SilkS)
-    (effects (font (size 0.5 0.5) (thickness 0.125)))
-  )
-  (gr_text a0 (at 165.354 75.057) (layer F.SilkS)
-    (effects (font (size 0.5 0.5) (thickness 0.125)))
-  )
-  (gr_text a0 (at 162.814 75.057) (layer F.SilkS)
-    (effects (font (size 0.5 0.5) (thickness 0.125)))
-  )
-  (gr_text a0 (at 160.274 75.057) (layer F.SilkS)
-    (effects (font (size 0.5 0.5) (thickness 0.125)))
-  )
-  (gr_text a0 (at 157.734 75.057) (layer F.SilkS)
-    (effects (font (size 0.5 0.5) (thickness 0.125)))
-  )
-  (gr_text a0 (at 155.194 75.057) (layer F.SilkS)
-    (effects (font (size 0.5 0.5) (thickness 0.125)))
-  )
-  (gr_text a0 (at 155.194 81.153) (layer F.SilkS)
-    (effects (font (size 0.5 0.5) (thickness 0.125)))
-  )
-  (gr_text a0 (at 157.734 81.153) (layer F.SilkS)
-    (effects (font (size 0.5 0.5) (thickness 0.125)))
-  )
-  (gr_text a0 (at 160.274 81.153) (layer F.SilkS)
-    (effects (font (size 0.5 0.5) (thickness 0.125)))
-  )
-  (gr_text a0 (at 162.814 81.153) (layer F.SilkS)
-    (effects (font (size 0.5 0.5) (thickness 0.125)))
-  )
-  (gr_text a0 (at 165.354 81.153) (layer F.SilkS)
-    (effects (font (size 0.5 0.5) (thickness 0.125)))
-  )
-  (gr_text a0 (at 167.894 81.153) (layer F.SilkS)
-    (effects (font (size 0.5 0.5) (thickness 0.125)))
-  )
-  (gr_text a0 (at 170.434 81.153) (layer F.SilkS)
+  (gr_text a1 (at 172.974 75.057) (layer F.SilkS)
+    (effects (font (size 0.5 0.5) (thickness 0.125)))
+  )
+  (gr_text "a3\n" (at 170.434 75.057) (layer F.SilkS)
+    (effects (font (size 0.5 0.5) (thickness 0.125)))
+  )
+  (gr_text a5 (at 167.894 75.057) (layer F.SilkS)
+    (effects (font (size 0.5 0.5) (thickness 0.125)))
+  )
+  (gr_text a7 (at 165.354 75.057) (layer F.SilkS)
+    (effects (font (size 0.5 0.5) (thickness 0.125)))
+  )
+  (gr_text a9 (at 162.814 75.057) (layer F.SilkS)
+    (effects (font (size 0.5 0.5) (thickness 0.125)))
+  )
+  (gr_text a11 (at 160.274 75.057) (layer F.SilkS)
+    (effects (font (size 0.5 0.5) (thickness 0.125)))
+  )
+  (gr_text a13 (at 157.734 75.057) (layer F.SilkS)
+    (effects (font (size 0.5 0.5) (thickness 0.125)))
+  )
+  (gr_text a15 (at 155.194 75.057) (layer F.SilkS)
+    (effects (font (size 0.5 0.5) (thickness 0.125)))
+  )
+  (gr_text a14 (at 155.194 81.153) (layer F.SilkS)
+    (effects (font (size 0.5 0.5) (thickness 0.125)))
+  )
+  (gr_text "a12\n" (at 157.734 81.153) (layer F.SilkS)
+    (effects (font (size 0.5 0.5) (thickness 0.125)))
+  )
+  (gr_text a10 (at 160.274 81.153) (layer F.SilkS)
+    (effects (font (size 0.5 0.5) (thickness 0.125)))
+  )
+  (gr_text a8 (at 162.814 81.153) (layer F.SilkS)
+    (effects (font (size 0.5 0.5) (thickness 0.125)))
+  )
+  (gr_text "a6\n" (at 165.354 81.153) (layer F.SilkS)
+    (effects (font (size 0.5 0.5) (thickness 0.125)))
+  )
+  (gr_text "a4\n" (at 167.894 81.153) (layer F.SilkS)
+    (effects (font (size 0.5 0.5) (thickness 0.125)))
+  )
+  (gr_text a2 (at 170.434 81.153) (layer F.SilkS)
     (effects (font (size 0.5 0.5) (thickness 0.125)))
   )
@@
     (effects (font (size 1 1) (thickness 0.15)))
   )
-  (gr_text "PWR I/O" (at 133.604 82.042) (layer F.SilkS)
+  (gr_text "PWR I/O" (at 133.604 82.677) (layer F.SilkS)
     (effects (font (size 1 1) (thickness 0.15)))
   )

Commit message: gitignore update + new button footprint name.
Connections:
- U4 pad 14: /+5V -> (no net)
- U4 pad 7: /GND -> (no net)
Changed lines of the file:
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@@
   )
   (setup
-    (last_trace_width 0.2)
+    (last_trace_width 0.5)
     (user_trace_width 0.2)
     (user_trace_width 0.25)
@@
     (pad 6 smd rect (at -2.90576 2.6416) (size 1.18 0.58) (layers F.Cu F.Paste F.Mask)
       (net 71 /NAND1))
-    (pad 7 smd rect (at -2.90576 3.9116) (size 1.18 0.58) (layers F.Cu F.Paste F.Mask)
-      (net 67 /GND))
+    (pad 7 smd rect (at -2.90576 3.9116) (size 1.18 0.58) (layers F.Cu F.Paste F.Mask))
     (pad 8 smd rect (at 3.15722 3.9116) (size 1.18 0.58) (layers F.Cu F.Paste F.Mask)
       (net 69 /#CS2))
@@
     (pad 13 smd rect (at 3.15722 -2.4384) (size 1.18 0.58) (layers F.Cu F.Paste F.Mask)
       (net 50 /CLK))
-    (pad 14 smd rect (at 3.15722 -3.7084) (size 1.18 0.58) (layers F.Cu F.Paste F.Mask)
-      (net 68 /+5V))
+    (pad 14 smd rect (at 3.15722 -3.7084) (size 1.18 0.58) (layers F.Cu F.Paste F.Mask))
   )
   (module Capacitor_SMD:C_1206_3216Metric_Pad1.42x1.75mm_HandSolder (layer B.Cu)
