File: design/board.kicad_pcb (KiCad board)
At the start: 2 copper layers, 165 x 54 mm, 22 parts, among them J1 Conn_01x04_Male, J2 Conn_01x03_Male, J3 Conn_02x14_Odd_Even, J4 Conn_02x12_Odd_Even, SW1 reset, U1 W65C02_PLCC_44, U2 AT28C256_PDIP_28, U3 SRAM, U4 74LS00, U5 2-AND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

Commit message: Better reset switch.
Parts:
- SW1: footprint my_buttons:pushbutton_button -> my_buttons:pushbutton_switch
- moved SW1 8.05 mm to (109.4, 71.5)
Routing:
- net /#RES: track 135.7 -> 141.3 mm
- net /#DMA: track 106.2 -> 103.6 mm
- net /GND: track 194.7 -> 193.9 mm, vias 10 -> 11
